File: SuperSocket16-ESP12F.kicad_pcb (KiCad board)
At the start: 2 copper layers, 90 x 40 mm, 25 parts, among them J1 Conn_01x08, J2 Conn_01x08, J3 Conn_02x10_Counter_Clockwise, J4 Conn_02x04, J5 Conn_01x08, J6 Conn_01x08, J7 Conn_02x04, J9 Conn_02x03, SW1 Reset, SW2 Program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

Commit message: Should be fully wired now. Fixed some mistakes pertaining to voltages.
Parts:
- J9: value Conn_02x03 -> Conn_02x02; footprint Connector_PinHeader_2.54mm:PinHeader_2x03_P2.54mm_Vertical -> Connector_PinHeader_2.54mm:PinHeader_2x02_P2.54mm_Vertical
- moved SW1 13.5 mm to (100.8, 101.9)
- moved SW2 13.4 mm to (94.3, 89.0)
- moved C1 10.4 mm to (106.0, 97.3)
- moved R1 10.4 mm to (113.5, 101.1)
- moved R2 10.4 mm to (113.5, 104.6)
- moved R4 10.4 mm to (113.5, 93.5)
- moved R5 10.4 mm to (105.9, 89.9)
- moved R6 10.4 mm to (113.5, 86.4)
- moved C3 2.57 mm to (122.6, 88.3), turned to 180 degrees
- moved J9 2.29 mm to (139.7, 109.7)
- moved U2 2.03 mm to (121.7, 96.5)
- moved C2 1.94 mm to (121.3, 103.5)
Connections:
- J9 pad 2: +5V -> +3V3
- J9 pad 4: +5V -> +3V3
- R7 pad 1: +5V -> +3V3
- R8 pad 1: +5V -> +3V3
- U3 pad 24: +5V -> +3V3
Routing:
- net +3V3: track 86.0 -> 135.1 mm
- net +5V: track 89.3 -> 40.7 mm
- net EN: track 24.1 -> 34.5 mm
- net GPIO15: track 18.6 -> 28.8 mm
- net GPIO0: track 44.7 -> 34.9 mm
- net INT#: track 75.5 -> 68.3 mm
- net RST: track 58.0 -> 51.3 mm
- net GND: track 150.8 -> 146.1 mm
- net Net-(J6-Pad2): track 8.49 -> 9.06 mm
Other:
- board text added: "Program"
- board text added: "Reset"
